File: Power_USB.kicad_sch (KiCad schematic)
At the start: 7 parts, among them J1 USB_C_Receptacle_USB2.0, U1 NCP1117-3.3_SOT223, U2 USBLC6-2P6

Commit message: Fixed duplicate annotations
Parts:
- renumbered C1 to C3, U1 to U2, U2 to U3
Other:
- note removed: "Optional USB-A for dongles?"
Changed lines of the file:
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@@
-    (effects (font (size 1.27 1.27)) (justify left bottom))
-  )
-  (text "Optional USB-A for dongles?" (at 174.625 38.1 0)
     (effects (font (size 1.27 1.27)) (justify left bottom))
   )
@@
   (symbol (lib_id "power:GND") (at 108.585 57.785 0) (unit 1)
     (in_bom yes) (on_board yes) (fields_autoplaced)
-    (property "Reference" "#PWR04" (id 0) (at 108.585 64.135 0)
+    (property "Reference" "#PWR0104" (id 0) (at 108.585 64.135 0)
       (effects (font (size 1.27 1.27)) hide)
     )
@@
   (symbol (lib_id "Power_Protection:USBLC6-2P6") (at 134.62 89.535 0) (unit 1)
     (in_bom yes) (on_board yes) (fields_autoplaced)
-    (property "Reference" "U2" (id 0) (at 137.3887 76.2 0)
+    (property "Reference" "U3" (id 0) (at 137.3887 76.2 0)
       (effects (font (size 1.27 1.27)) (justify left))
     )
@@
   (symbol (lib_id "power:GND") (at 76.835 88.265 0) (unit 1)
     (in_bom yes) (on_board yes) (fields_autoplaced)
-    (property "Reference" "#PWR02" (id 0) (at 76.835 94.615 0)
+    (property "Reference" "#PWR0101" (id 0) (at 76.835 94.615 0)
       (effects (font (size 1.27 1.27)) hide)
     )
@@
   (symbol (lib_id "power:GND") (at 69.215 88.265 0) (unit 1)
     (in_bom yes) (on_board yes) (fields_autoplaced)
-    (property "Reference" "#PWR01" (id 0) (at 69.215 94.615 0)
+    (property "Reference" "#PWR0102" (id 0) (at 69.215 94.615 0)
       (effects (font (size 1.27 1.27)) hide)
     )
@@
   (symbol (lib_id "power:GND") (at 114.935 55.245 0) (unit 1)
     (in_bom yes) (on_board yes) (fields_autoplaced)
-    (property "Reference" "#PWR05" (id 0) (at 114.935 61.595 0)
+    (property "Reference" "#PWR0109" (id 0) (at 114.935 61.595 0)
       (effects (font (size 1.27 1.27)) hide)
     )
@@
   (symbol (lib_id "power:VBUS") (at 92.075 50.165 0) (unit 1)
     (in_bom yes) (on_board yes)
-    (property "Reference" "#PWR03" (id 0) (at 92.075 53.975 0)
+    (property "Reference" "#PWR0103" (id 0) (at 92.075 53.975 0)
       (effects (font (size 1.27 1.27)) hide)
     )
@@
   (symbol (lib_id "Device:C_Small") (at 114.935 52.705 0) (unit 1)
     (in_bom yes) (on_board yes) (fields_autoplaced)
-    (property "Reference" "C1" (id 0) (at 118.11 51.4412 0)
+    (property "Reference" "C3" (id 0) (at 118.11 51.4412 0)
       (effects (font (size 1.27 1.27)) (justify left))
     )
@@
   (symbol (lib_id "Regulator_Linear:NCP1117-3.3_SOT223") (at 127.635 50.165 0) (unit 1)
     (in_bom yes) (on_board yes) (fields_autoplaced)
-    (property "Reference" "U1" (id 0) (at 127.635 43.18 0))
+    (property "Reference" "U2" (id 0) (at 127.635 43.18 0))
     (property "Value" "NCP1117-3.3_SOT223" (id 1) (at 127.635 45.72 0))
     (property "Footprint" "Package_TO_SOT_SMD:SOT-223-3_TabPin2" (id 2) (at 127.635 45.085 0)
@@
   (symbol (lib_id "power:GND") (at 127.635 57.785 0) (unit 1)
     (in_bom yes) (on_board yes) (fields_autoplaced)
-    (property "Reference" "#PWR06" (id 0) (at 127.635 64.135 0)
-      (effects (font (size 1.27 1.27)) hide)
-    )
+    (property "Reference" "#PWR0110" (id 0) (at 127.635 64.135 0)
+      (effects (font (size 1.27 1.27)) hide)
+    )
